File: kicad/pico_remote_sensor.kicad_pcb (KiCad board)
At the start: 2 copper layers, 39.9 x 54.9 mm, 15 parts, among them J1 Conn_02x20_Counter_Clockwise, J2 Conn_02x20_Counter_Clockwise, U1 Pico, U2 RFM75

Commit message: Board versions added
Other:
- board text added: "B r${version}"
- board text added: "F r${version}"
Changed lines of the file:
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@@
   (gr_line (start 134.62 84.678874) (end 134.62 84.678874) (layer "Edge.Cuts") (width 0.145018))
   (gr_line (start 134.62 29.823893) (end 134.62 29.823893) (layer "Edge.Cuts") (width 0.145018))
+  (gr_text "F r${version}" (at 99.427295 62.76673) (layer "F.Cu")
+    (effects (font (size 1 1) (thickness 0.2)))
+  )
+  (gr_text "B r${version}" (at 99.845019 71.978874) (layer "B.Cu")
+    (effects (font (size 1 1) (thickness 0.2)) (justify mirror))
+  )
   (via (at 134.765019 29.678874) (size 2) (drill 0.9) (layers "F.Cu" "B.Cu") (free) (net 0))
   (via (at 94.765019 84.678874) (size 2) (drill 0.9) (layers "F.Cu" "B.Cu") (free) (net 0))
